File: Hardware/USB-DALI.kicad_sch (KiCad schematic)
At the start: 43 parts, among them J1 USB_A, J2 ST-LINK, J3 Screw_Terminal_01x02, J4 PWR DALI BUS +, J5 PWR DALI BUS -, Q1 BCX56, U1 STM32F103C8T6, U2 PC817, U3 PC817, U4 AMS1117-3.3, U5 MT3608, Y1 8MHz

Commit message: Schematics in pdf and link to win driver added
Other:
- title: (none) -> https://github.com/even-notodd/USB-DALI
Changed lines of the file:
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@@
 	(generator_version "8.0")
 	(paper "A4")
+	(title_block
+		(title "https://github.com/even-notodd/USB-DALI")
+	)
 	(junction
 		(at 233.68 135.89)
